File: nagmtly2026-board-esp32-solo-1-v1.0.kicad_sch (KiCad schematic)
At the start: 0 parts

Commit message: update: 回路図を更新(Apr 02:56)
Parts:
- added C6, C7: 0.1u, symbol Device:C
- added J2, J3: Conn_01x20, symbol Connector_Generic:Conn_01x20
- added R8: 470, symbol Device:R
- added SW1, SW2: SW_Push, symbol Switch:SW_Push
Connections:
- new net +3.3VS: J2.1 (Pin_1)
- new net EN: C6.1, J2.2 (Pin_2), SW1.2
- new net GNDS: C6.2, C7.2, J2.20 (Pin_20), J2.9 (Pin_9), J3.1 (Pin_1), J3.9 (Pin_9), SW1.1, SW2.1
- new net IO0: C7.1, SW2.2
- new net IO12: J2.7 (Pin_7)
- new net IO13: J2.8 (Pin_8)
- new net IO14: J2.6 (Pin_6)
- new net IO15: J2.5 (Pin_5)
- new net IO19: J3.8 (Pin_8)
- new net IO21: J3.5 (Pin_5)
- new net IO23: J3.2 (Pin_2)
- new net IO25: J2.3 (Pin_3)
- new net IO26: J2.4 (Pin_4)
- new net IO27: J2.10 (Pin_10)
- new net IO4: J3.3 (Pin_3)
- new net MCU/ESP32_RXD: R8.1
- new net SENSOR_VN: J2.19 (Pin_19)
- new net SENSOR_VP: J2.18 (Pin_18)
- new net USB/FT232_TXD: R8.2
- no-connect marks 0 -> 10
Other:
- added sheet MCU (ESP32-SOLO-1.kicad_sch)
- added sheet USB (FT231XS.kicad_sch)
